File: docs/LX790_V1_1/Adapter Cable.kicad_sch (KiCad schematic)
At the start: 6 parts

Commit message: update documentation
Connections:
- net at J?.10 (Pin_10), J?.10 (Pin_10): no longer J?.11 (Pin_11)
- net at J?.9 (Pin_9), J?.9 (Pin_9): now also J?.11 (Pin_11)
Changed lines of the file:
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@@
   (junction (at 77.47 122.555) (diameter 0) (color 0 0 0 0)
   )
+  (junction (at 182.88 64.135) (diameter 0) (color 0 0 0 0)
+  )
   (junction (at 151.13 97.155) (diameter 0) (color 0 0 0 0)
   )
@@
   (junction (at 77.47 51.435) (diameter 0) (color 0 0 0 0)
   )
-  (junction (at 182.88 66.675) (diameter 0) (color 0 0 0 0)
-  )
   (junction (at 170.18 74.295) (diameter 0) (color 0 0 0 0)
   )
@@
     (stroke (width 0) (type default) (color 0 0 0 0))
   )
-  (wire (pts (xy 41.91 64.135) (xy 189.23 64.135))
-    (stroke (width 0) (type default) (color 0 0 0 0))
-  )
-  (wire (pts (xy 182.88 66.675) (xy 189.23 66.675))
+  (wire (pts (xy 41.91 64.135) (xy 182.88 64.135))
     (stroke (width 0) (type default) (color 0 0 0 0))
   )
@@
     (stroke (width 0) (type default) (color 0 0 0 0))
   )
+  (wire (pts (xy 182.88 64.135) (xy 189.23 64.135))
+    (stroke (width 0) (type default) (color 0 0 0 0))
+  )
   (wire (pts (xy 41.91 51.435) (xy 77.47 51.435))
     (stroke (width 0) (type default) (color 0 0 0 0))
@@
     (stroke (width 0) (type default) (color 0 0 0 0))
   )
+  (wire (pts (xy 182.88 64.135) (xy 182.88 69.215))
+    (stroke (width 0) (type default) (color 0 0 0 0))
+  )
   (wire (pts (xy 106.68 122.555) (xy 102.87 122.555))
     (stroke (width 0) (type default) (color 0 0 0 0))
@@
     (stroke (width 0) (type default) (color 0 0 0 0))
   )
-  (wire (pts (xy 41.91 66.675) (xy 182.88 66.675))
+  (wire (pts (xy 41.91 66.675) (xy 189.23 66.675))
     (stroke (width 0) (type default) (color 0 0 0 0))
   )
@@
     (stroke (width 0) (type default) (color 0 0 0 0))
   )
-  (wire (pts (xy 182.88 69.215) (xy 182.88 66.675))
-    (stroke (width 0) (type default) (color 0 0 0 0))
-  )

Commit message: add NTP time
Connections:
- net at J?.1 (Pin_1), J?.1 (Pin_1): now also R?.1
- net VCC: no longer names the net of D?.1 (K), X?.1 (Vin)
- net VCC: no longer R?.1
Changed lines of the file:
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@@
   (junction (at 182.88 64.135) (diameter 0) (color 0 0 0 0)
   )
-  (junction (at 151.13 97.155) (diameter 0) (color 0 0 0 0)
-  )
-  (junction (at 135.255 97.155) (diameter 0) (color 0 0 0 0)
+  (junction (at 106.68 43.815) (diameter 0) (color 0 0 0 0)
   )
   (junction (at 116.84 79.375) (diameter 0) (color 0 0 0 0)
@@
   (junction (at 173.99 81.915) (diameter 0) (color 0 0 0 0)
   )
-  (wire (pts (xy 106.68 104.775) (xy 106.68 97.155))
-    (stroke (width 0) (type default) (color 0 0 0 0))
-  )
   (wire (pts (xy 147.32 107.315) (xy 151.13 107.315))
     (stroke (width 0) (type default) (color 0 0 0 0))
@@
     (stroke (width 0) (type default) (color 0 0 0 0))
   )
-  (wire (pts (xy 151.13 92.075) (xy 151.13 97.155))
-    (stroke (width 0) (type default) (color 0 0 0 0))
-  )
   (wire (pts (xy 158.75 112.395) (xy 158.75 56.515))
     (stroke (width 0) (type default) (color 0 0 0 0))
@@
     (stroke (width 0) (type default) (color 0 0 0 0))
   )
-  (wire (pts (xy 135.255 97.155) (xy 151.13 97.155))
-    (stroke (width 0) (type default) (color 0 0 0 0))
-  )
   (wire (pts (xy 87.63 117.475) (xy 82.55 117.475))
     (stroke (width 0) (type default) (color 0 0 0 0))
   )
-  (wire (pts (xy 151.13 107.315) (xy 151.13 97.155))
-    (stroke (width 0) (type default) (color 0 0 0 0))
-  )
-  (wire (pts (xy 41.91 43.815) (xy 189.23 43.815))
+  (wire (pts (xy 151.13 92.075) (xy 151.13 107.315))
+    (stroke (width 0) (type default) (color 0 0 0 0))
+  )
+  (wire (pts (xy 41.91 43.815) (xy 106.68 43.815))
     (stroke (width 0) (type default) (color 0 0 0 0))
   )
@@
     (stroke (width 0) (type default) (color 0 0 0 0))
   )
+  (wire (pts (xy 106.68 43.815) (xy 189.23 43.815))
+    (stroke (width 0) (type default) (color 0 0 0 0))
+  )
   (wire (pts (xy 186.69 122.555) (xy 186.69 69.215))
     (stroke (width 0) (type default) (color 0 0 0 0))
@@
     (stroke (width 0) (type default) (color 0 0 0 0))
   )
-  (wire (pts (xy 135.255 92.71) (xy 135.255 97.155))
-    (stroke (width 0) (type default) (color 0 0 0 0))
-  )
-  (wire (pts (xy 106.68 97.155) (xy 135.255 97.155))
+  (wire (pts (xy 106.68 43.815) (xy 106.68 104.775))
     (stroke (width 0) (type default) (color 0 0 0 0))
   )
@@
     (pin "2")
   )
-  (symbol (lib_id "power:VCC") (at 135.255 92.71 0) (unit 1)
-    (in_bom yes) (on_board yes)
-    (property "Reference" "#PWR?" (id 0) (at 135.255 96.52 0)
-      (effects (font (size 1.27 1.27)) hide)
-    )
-    (property "Value" "VCC" (id 1) (at 131.445 90.805 0))
-    (property "Footprint" "" (id 2) (at 135.255 92.71 0)
-      (effects (font (size 1.27 1.27)) hide)
-    )
-    (property "Datasheet" "" (id 3) (at 135.255 92.71 0)
-      (effects (font (size 1.27 1.27)) hide)
-    )
-    (pin "1")
-  )
   (sheet_instances
     (path "/" (page "1"))
@@
       (reference "#PWR?") (unit 1) (value "GNDD") (footprint "")
     )
-    (path "/fc1cf631-2e5a-4ee6-bcc1-950e14bf50c4"
-      (reference "#PWR?") (unit 1) (value "VCC") (footprint "")
-    )
     (path "/e28efe3d-8d67-44a7-9f24-6996853c174e"
